Commit message: add simple collision conditionals in URDF files

File: ros2_humanoid_virtual_twin/description/RobotElements/LeftLegElems/Lankle.xacro (robot description, xacro)
@@ -19,10 +19,20 @@
         <material name="grey"/>
       </visual>
-      <collision>
-        <origin xyz="0 0 0" rpy="0 0 0"/>
-        <geometry>
+      <xacro:if value="$(arg use_simple_collision)">
+        <collision>
+          <origin xyz="-0.022 0.003 0.0168" rpy="0 0 0"/>
+          <geometry>
+            <box size="0.101 0.05 0.0626"/>
+          </geometry>
+        </collision>
+      </xacro:if>
+      <xacro:unless value="$(arg use_simple_collision)">
+        <collision>
+          <origin xyz="0 0 0" rpy="0 0 0"/>
+          <geometry>
             <mesh filename="file://$(find ros2_humanoid_virtual_twin)/meshes/Left-Ankle-Collision.stl"/>
-        </geometry>
-      </collision>
+          </geometry>
+        </collision>
+      </xacro:unless>
       <inertial>
         <origin xyz="-20.881e-3	0.167e-3	14.849e-3" rpy="0 0 0"/>

File: ros2_humanoid_virtual_twin/description/RobotElements/LeftLegElems/Lfoot.xacro (robot description, xacro)
@@ -20,10 +20,20 @@
         <material name="grey"/>
       </visual>
-      <collision>
-        <origin xyz="0 0 0" rpy="0 0 0"/>
-        <geometry>
-			    <mesh filename="file://$(find ros2_humanoid_virtual_twin)/meshes/Left-Foot-collision.stl"/>
-        </geometry>
-      </collision>
+      <xacro:if value="$(arg use_simple_collision)">
+        <collision>
+          <origin xyz="-0.003 0 -0.01200198" rpy="0 0 0"/>
+          <geometry>
+            <box size="0.134 0.072 0.05199603"/>
+          </geometry>
+        </collision>
+      </xacro:if>
+      <xacro:unless value="$(arg use_simple_collision)">
+        <collision>
+          <origin xyz="0 0 0" rpy="0 0 0"/>
+          <geometry>
+            <mesh filename="file://$(find ros2_humanoid_virtual_twin)/meshes/Left-Foot-collision.stl"/>
+          </geometry>
+        </collision>
+      </xacro:unless>
       <inertial>
         <origin xyz="-5.077e-3	0	-30.402e-3" rpy="0 0 0"/>

File: ros2_humanoid_virtual_twin/description/RobotElements/LeftLegElems/Lhip.xacro (robot description, xacro)
@@ -20,10 +20,20 @@
         <material name="grey"/>
       </visual>
-      <collision>
-        <origin xyz="0 0 0" rpy="0 0 0"/>
-        <geometry>
+      <xacro:if value="$(arg use_simple_collision)">
+        <collision>
+          <origin xyz="-0.022 -0.003 -0.0168" rpy="0 0 0"/>
+          <geometry>
+            <box size="0.101 0.05 0.0626"/>
+          </geometry>
+        </collision>
+      </xacro:if>
+      <xacro:unless value="$(arg use_simple_collision)">
+        <collision>
+          <origin xyz="0 0 0" rpy="0 0 0"/>
+          <geometry>
             <mesh filename="file://$(find ros2_humanoid_virtual_twin)/meshes/Right-Hip-Collision.stl"/>
-        </geometry>
-      </collision>
+          </geometry>
+        </collision>
+      </xacro:unless>
       <inertial>
         <origin xyz="-20.881e-3	-0.167e-3	-14.849e-3" rpy="0 0 0"/>

File: ros2_humanoid_virtual_twin/description/RobotElements/LeftLegElems/Lhipmount.xacro (robot description, xacro)
@@ -21,10 +21,20 @@
       <material name="grey"/>
     </visual>
-    <collision>
-      <origin xyz="0 0 0" rpy="0 0 0"/>
-      <geometry>
-        <mesh filename="file://$(find ros2_humanoid_virtual_twin)/meshes/Rgiht-HipMount-Collision.stl"/>
-      </geometry>
-    </collision>
+    <xacro:if value="$(arg use_simple_collision)">
+      <collision>
+        <origin xyz="-0.019 0 0.01100793" rpy="0 0 0"/>
+        <geometry>
+          <box size="0.102 0.036 0.04998414"/>
+        </geometry>
+      </collision>
+    </xacro:if>
+    <xacro:unless value="$(arg use_simple_collision)">
+      <collision>
+        <origin xyz="0 0 0" rpy="0 0 0"/>
+        <geometry>
+          <mesh filename="file://$(find ros2_humanoid_virtual_twin)/meshes/Right-HipMount-Collision.stl"/>
+        </geometry>
+      </collision>
+    </xacro:unless>
     <inertial>
       <origin xyz="-13.999e-3	0	24.592e-3" rpy="0 0 0"/>

File: ros2_humanoid_virtual_twin/description/RobotElements/LeftLegElems/Lshank.xacro (robot description, xacro)
@@ -19,10 +19,20 @@
         <material name="grey"/>
       </visual>
-      <collision>
-        <origin xyz="0 0 0" rpy="0 0 0"/>
-        <geometry>
+      <xacro:if value="$(arg use_simple_collision)">
+        <collision>
+          <origin xyz="0.0035 0 -0.064" rpy="0 0 0"/>
+          <geometry>
+            <box size="0.035 0.051 0.15599208"/>
+          </geometry>
+        </collision>
+      </xacro:if>
+      <xacro:unless value="$(arg use_simple_collision)">
+        <collision>
+          <origin xyz="0 0 0" rpy="0 0 0"/>
+          <geometry>
             <mesh filename="file://$(find ros2_humanoid_virtual_twin)/meshes/Right-Shank-Collision.stl"/>
-        </geometry>
-      </collision>
+          </geometry>
+        </collision>
+      </xacro:unless>
       <inertial>
         <origin xyz="4.836e-3	-2.813e-3	-60.226e-3" rpy="0 0 0"/>

File: ros2_humanoid_virtual_twin/description/RobotElements/LeftLegElems/Lthigh.xacro (robot description, xacro)
@@ -19,10 +19,20 @@
         <material name="grey"/>
       </visual>
-      <collision>
-        <origin xyz="0 0 0" rpy="0 0 0"/>
-        <geometry>
+      <xacro:if value="$(arg use_simple_collision)">
+        <collision>
+          <origin xyz="0.00295 0.00125 -0.06400793" rpy="0 0 0"/>
+          <geometry>
+            <box size="0.0461 0.0535 0.15598415"/>
+          </geometry>
+        </collision>
+      </xacro:if>
+      <xacro:unless value="$(arg use_simple_collision)">
+        <collision>
+          <origin xyz="0 0 0" rpy="0 0 0"/>
+          <geometry>
             <mesh filename="file://$(find ros2_humanoid_virtual_twin)/meshes/Right-Thigh-Collision.stl"/>
-        </geometry>
-      </collision>
+          </geometry>
+        </collision>
+      </xacro:unless>
       <inertial>
         <origin xyz="2.704e-3	0.696e-3 -97.695e-3" rpy="0 0 0"/>

File: ros2_humanoid_virtual_twin/description/RobotElements/RightLegElems/Rankle.xacro (robot description, xacro)
@@ -15,16 +15,24 @@
             <origin xyz="0 0 0" rpy="0 0 0"/>
             <geometry>
-                <!-- Left ankle is used to describe right ankle because visually they're the same -->
                 <mesh filename="file://$(find ros2_humanoid_virtual_twin)/meshes/Left-Ankle.stl"/>
             </geometry>
             <material name="grey"/>
         </visual>
-        <collision>
-            <origin xyz="0 0 0" rpy="0 0 0"/>
-            <geometry>
-                <!-- Left ankle is used to describe right ankle because visually they're the same -->
+        <xacro:if value="$(arg use_simple_collision)">
+            <collision>
+                <origin xyz="-0.022 0.003 0.0168" rpy="0 0 0"/>
+                <geometry>
+                <box size="0.101 0.05 0.0626"/>
+                </geometry>
+            </collision>
+            </xacro:if>
+            <xacro:unless value="$(arg use_simple_collision)">
+            <collision>
+                <origin xyz="0 0 0" rpy="0 0 0"/>
+                <geometry>
                 <mesh filename="file://$(find ros2_humanoid_virtual_twin)/meshes/Left-Ankle-Collision.stl"/>
-            </geometry>
-        </collision>
+                </geometry>
+            </collision>
+        </xacro:unless>
         <inertial>
             <origin xyz="-20.881e-3	0.167e-3 14.849e-3" rpy="0 0 0"/>

File: ros2_humanoid_virtual_twin/description/RobotElements/RightLegElems/Rfoot.xacro (robot description, xacro)
@@ -19,10 +19,20 @@
             <material name="grey"/>
         </visual>
-        <collision>
+        <xacro:if value="$(arg use_simple_collision)">
+            <collision>
+            <origin xyz="-0.003 0 -0.01200198" rpy="0 0 0"/>
+            <geometry>
+                <box size="0.134 0.072 0.05199603"/>
+            </geometry>
+            </collision>
+        </xacro:if>
+        <xacro:unless value="$(arg use_simple_collision)">
+            <collision>
             <origin xyz="0 0 0" rpy="0 0 0"/>
             <geometry>
                 <mesh filename="file://$(find ros2_humanoid_virtual_twin)/meshes/Left-Foot-collision.stl"/>
             </geometry>
-        </collision>
+            </collision>
+        </xacro:unless>
         <inertial>
             <origin xyz="-5.077e-3	0	-30.402e-3" rpy="0 0 0"/>

File: ros2_humanoid_virtual_twin/description/RobotElements/RightLegElems/Rhip.xacro (robot description, xacro)
@@ -19,10 +19,20 @@
             <material name="grey"/>
         </visual>
-        <collision>
+        <xacro:if value="$(arg use_simple_collision)">
+            <collision>
+            <origin xyz="-0.022 -0.003 -0.0168" rpy="0 0 0"/>
+            <geometry>
+                <box size="0.101 0.05 0.0626"/>
+            </geometry>
+            </collision>
+        </xacro:if>
+        <xacro:unless value="$(arg use_simple_collision)">
+            <collision>
             <origin xyz="0 0 0" rpy="0 0 0"/>
             <geometry>
                 <mesh filename="file://$(find ros2_humanoid_virtual_twin)/meshes/Right-Hip-Collision.stl"/>
             </geometry>
-        </collision>
+            </collision>
+        </xacro:unless>
         <inertial>
             <origin xyz="-20.881e-3	-0.167e-3	-14.849e-3" rpy="0 0 0"/>

File: ros2_humanoid_virtual_twin/description/RobotElements/RightLegElems/Rhipmount.xacro (robot description, xacro)
@@ -19,10 +19,20 @@
             <material name="grey"/>
         </visual>
-        <collision>
-            <origin xyz="0 0 0" rpy="0 0 0"/>
-            <geometry>
+        <xacro:if value="$(arg use_simple_collision)">
+            <collision>
+                <origin xyz="-0.019 0 0.01100793" rpy="0 0 0"/>
+                <geometry>
+                <box size="0.102 0.036 0.04998414"/>
+                </geometry>
+            </collision>
+            </xacro:if>
+            <xacro:unless value="$(arg use_simple_collision)">
+            <collision>
+                <origin xyz="0 0 0" rpy="0 0 0"/>
+                <geometry>
                 <mesh filename="file://$(find ros2_humanoid_virtual_twin)/meshes/Right-HipMount-Collision.stl"/>
-            </geometry>
-        </collision>
+                </geometry>
+            </collision>
+        </xacro:unless>
         <inertial>
             <origin xyz="-13.999e-3	0	24.592e-3" rpy="0 0 0"/>

File: ros2_humanoid_virtual_twin/description/RobotElements/RightLegElems/Rshank.xacro (robot description, xacro)
@@ -19,10 +19,20 @@
             <material name="grey"/>
         </visual>
-        <collision>
+        <xacro:if value="$(arg use_simple_collision)">
+            <collision>
+            <origin xyz="0.0035 0 -0.064" rpy="0 0 0"/>
+            <geometry>
+                <box size="0.035 0.051 0.15599208"/>
+            </geometry>
+            </collision>
+        </xacro:if>
+        <xacro:unless value="$(arg use_simple_collision)">
+            <collision>
             <origin xyz="0 0 0" rpy="0 0 0"/>
             <geometry>
                 <mesh filename="file://$(find ros2_humanoid_virtual_twin)/meshes/Right-Shank-Collision.stl"/>
             </geometry>
-        </collision>
+            </collision>
+        </xacro:unless>
         <inertial>
             <origin xyz="4.836e-3	-2.813e-3	-60.226e-3" rpy="0 0 0"/>

File: ros2_humanoid_virtual_twin/description/RobotElements/RightLegElems/Rthigh.xacro (robot description, xacro)
@@ -19,10 +19,20 @@
             <material name="grey"/>
         </visual>
-        <collision>
+        <xacro:if value="$(arg use_simple_collision)">
+            <collision>
+            <origin xyz="0.00295 0.00125 -0.06400793" rpy="0 0 0"/>
+            <geometry>
+                <box size="0.0461 0.0535 0.15598415"/>
+            </geometry>
+            </collision>
+        </xacro:if>
+        <xacro:unless value="$(arg use_simple_collision)">
+            <collision>
             <origin xyz="0 0 0" rpy="0 0 0"/>
             <geometry>
                 <mesh filename="file://$(find ros2_humanoid_virtual_twin)/meshes/Right-Thigh-Collision.stl"/>
             </geometry>
-        </collision>
+            </collision>
+        </xacro:unless>
         <inertial>
             <origin xyz="2.704e-3	0.696e-3 -97.695e-3" rpy="0 0 0"/>

Commit message: update simplified collisions
Adjust primitive collision geometry to avoid self-collisions

File: ros2_humanoid_virtual_twin/description/RobotElements/LeftLegElems/Lankle.xacro (robot description, xacro)
@@ -21,7 +21,7 @@
       <xacro:if value="$(arg use_simple_collision)">
         <collision>
-          <origin xyz="-0.022 0.003 0.0168" rpy="0 0 0"/>
+          <origin xyz="-0.02 0.003 0.0168" rpy="0 0 0"/>
           <geometry>
-            <box size="0.101 0.05 0.0626"/>
+            <box size="0.106 0.05 0.063"/>
           </geometry>
         </collision>

File: ros2_humanoid_virtual_twin/description/RobotElements/LeftLegElems/Lfoot.xacro (robot description, xacro)
@@ -22,7 +22,7 @@
       <xacro:if value="$(arg use_simple_collision)">
         <collision>
-          <origin xyz="-0.003 0 -0.01200198" rpy="0 0 0"/>
+          <origin xyz="-0.003 0 -0.0325" rpy="0 0 0"/>
           <geometry>
-            <box size="0.134 0.072 0.05199603"/>
+            <box size="0.134 0.072 0.011"/>
           </geometry>
         </collision>

File: ros2_humanoid_virtual_twin/description/RobotElements/LeftLegElems/Lhip.xacro (robot description, xacro)
@@ -22,7 +22,7 @@
       <xacro:if value="$(arg use_simple_collision)">
         <collision>
-          <origin xyz="-0.022 -0.003 -0.0168" rpy="0 0 0"/>
+          <origin xyz="-0.02 -0.0013 -0.0168" rpy="0 0 0"/>
           <geometry>
-            <box size="0.101 0.05 0.0626"/>
+            <box size="0.105 0.0538 0.0626"/>
           </geometry>
         </collision>

File: ros2_humanoid_virtual_twin/description/RobotElements/LeftLegElems/Lhipmount.xacro (robot description, xacro)
@@ -23,7 +23,7 @@
     <xacro:if value="$(arg use_simple_collision)">
       <collision>
-        <origin xyz="-0.019 0 0.01100793" rpy="0 0 0"/>
+        <origin xyz="-0.019 0 0.0325" rpy="0 0 0"/>
         <geometry>
-          <box size="0.102 0.036 0.04998414"/>
+          <box size="0.102 0.036 0.007"/>
         </geometry>
       </collision>
@@ -33,5 +33,5 @@
         <origin xyz="0 0 0" rpy="0 0 0"/>
         <geometry>
-          <mesh filename="file://$(find ros2_humanoid_virtual_twin)/meshes/Right-HipMount-Collision.stl"/>
+          <mesh filename="file://$(find ros2_humanoid_virtual_twin)/meshes/Rgiht-HipMount-Collision.stl"/>
         </geometry>
       </collision>

File: ros2_humanoid_virtual_twin/description/RobotElements/LeftLegElems/Lshank.xacro (robot description, xacro)
@@ -21,7 +21,7 @@
       <xacro:if value="$(arg use_simple_collision)">
         <collision>
-          <origin xyz="0.0035 0 -0.064" rpy="0 0 0"/>
+          <origin xyz="0.0023 0 -0.033" rpy="0 0 0"/>
           <geometry>
-            <box size="0.035 0.051 0.15599208"/>
+            <box size="0.045 0.058 0.07"/>
           </geometry>
         </collision>

File: ros2_humanoid_virtual_twin/description/RobotElements/LeftLegElems/Lthigh.xacro (robot description, xacro)
@@ -21,7 +21,7 @@
       <xacro:if value="$(arg use_simple_collision)">
         <collision>
-          <origin xyz="0.00295 0.00125 -0.06400793" rpy="0 0 0"/>
+          <origin xyz="0.00295 0.00125 -0.081" rpy="0 0 0"/>
           <geometry>
-            <box size="0.0461 0.0535 0.15598415"/>
+            <box size="0.0461 0.0535 0.043"/>
           </geometry>
         </collision>

File: ros2_humanoid_virtual_twin/description/RobotElements/RightLegElems/Rankle.xacro (robot description, xacro)
@@ -21,7 +21,7 @@
         <xacro:if value="$(arg use_simple_collision)">
             <collision>
-                <origin xyz="-0.022 0.003 0.0168" rpy="0 0 0"/>
+                <origin xyz="-0.02 0.003 0.0168" rpy="0 0 0"/>
                 <geometry>
-                <box size="0.101 0.05 0.0626"/>
+                <box size="0.106 0.05 0.063"/>
                 </geometry>
             </collision>

File: ros2_humanoid_virtual_twin/description/RobotElements/RightLegElems/Rfoot.xacro (robot description, xacro)
@@ -20,19 +20,19 @@
         </visual>
         <xacro:if value="$(arg use_simple_collision)">
-            <collision>
-            <origin xyz="-0.003 0 -0.01200198" rpy="0 0 0"/>
-            <geometry>
-                <box size="0.134 0.072 0.05199603"/>
-            </geometry>
-            </collision>
-        </xacro:if>
-        <xacro:unless value="$(arg use_simple_collision)">
-            <collision>
-            <origin xyz="0 0 0" rpy="0 0 0"/>
-            <geometry>
-                <mesh filename="file://$(find ros2_humanoid_virtual_twin)/meshes/Left-Foot-collision.stl"/>
-            </geometry>
-            </collision>
-        </xacro:unless>
+        <collision>
+          <origin xyz="-0.003 0 -0.0325" rpy="0 0 0"/>
+          <geometry>
+            <box size="0.134 0.072 0.011"/>
+          </geometry>
+        </collision>
+      </xacro:if>
+      <xacro:unless value="$(arg use_simple_collision)">
+        <collision>
+          <origin xyz="0 0 0" rpy="0 0 0"/>
+          <geometry>
+            <mesh filename="file://$(find ros2_humanoid_virtual_twin)/meshes/Left-Foot-collision.stl"/>
+          </geometry>
+        </collision>
+      </xacro:unless>
         <inertial>
             <origin xyz="-5.077e-3	0	-30.402e-3" rpy="0 0 0"/>

File: ros2_humanoid_virtual_twin/description/RobotElements/RightLegElems/Rhip.xacro (robot description, xacro)
@@ -21,7 +21,7 @@
         <xacro:if value="$(arg use_simple_collision)">
             <collision>
-            <origin xyz="-0.022 -0.003 -0.0168" rpy="0 0 0"/>
+            <origin xyz="-0.02 -0.0013 -0.0168" rpy="0 0 0"/>
             <geometry>
-                <box size="0.101 0.05 0.0626"/>
+                <box size="0.105 0.0538 0.0626"/>
             </geometry>
             </collision>

File: ros2_humanoid_virtual_twin/description/RobotElements/RightLegElems/Rhipmount.xacro (robot description, xacro)
@@ -21,7 +21,7 @@
         <xacro:if value="$(arg use_simple_collision)">
             <collision>
-                <origin xyz="-0.019 0 0.01100793" rpy="0 0 0"/>
+                <origin xyz="-0.019 0 0.0325" rpy="0 0 0"/>
                 <geometry>
-                <box size="0.102 0.036 0.04998414"/>
+                <box size="0.102 0.036 0.007"/>
                 </geometry>
             </collision>

File: ros2_humanoid_virtual_twin/description/RobotElements/RightLegElems/Rshank.xacro (robot description, xacro)
@@ -21,7 +21,7 @@
         <xacro:if value="$(arg use_simple_collision)">
             <collision>
-            <origin xyz="0.0035 0 -0.064" rpy="0 0 0"/>
+            <origin xyz="0.0023 0 -0.033" rpy="0 0 0"/>
             <geometry>
-                <box size="0.035 0.051 0.15599208"/>
+                <box size="0.045 0.058 0.07"/>
             </geometry>
             </collision>

File: ros2_humanoid_virtual_twin/description/RobotElements/RightLegElems/Rthigh.xacro (robot description, xacro)
@@ -21,7 +21,7 @@
         <xacro:if value="$(arg use_simple_collision)">
             <collision>
-            <origin xyz="0.00295 0.00125 -0.06400793" rpy="0 0 0"/>
+            <origin xyz="0.00295 0.00125 -0.081" rpy="0 0 0"/>
             <geometry>
-                <box size="0.0461 0.0535 0.15598415"/>
+                <box size="0.0461 0.0535 0.043"/>
             </geometry>
             </collision>
